Commit message: target detect and command to joint

File: ros2_ws/src/robot_shooter/urdf/shooter_robot.urdf.xacro (robot description, xacro)
@@ -61,4 +61,7 @@
     <color rgba="0 0 0.8 1"/>
   </material>
+  <material name="yellow">
+    <color rgba="0.8 0.8 0 1"/>
+  </material>
 <!-- ROBOT CONSTRUCTION -->
   <!-- Robot Base Link -->
@@ -94,5 +97,5 @@
         <cylinder radius="${pan_link_radius}" length="${pan_link_length}"/>
       </geometry>
-      <!-- <material name="green"/> -->
+      <material name="yellow"/>
       <origin rpy="0 0 0" xyz="0 0 0"/>
     </visual>
@@ -115,4 +118,5 @@
       </geometry>
       <origin rpy="0 0 0" xyz="0 0 0"/>
+      <material name="blue"/>
     </visual>
     <collision>
@@ -122,4 +126,5 @@
       <origin xyz="0.0 0.0 0.0" rpy="0.0 0.0 0.0"/>
     </collision>
+    <material name="blue" />
   </link>
   <joint name="pan_to_right_pillar_joint" type="fixed">
@@ -134,4 +139,5 @@
       </geometry>
       <origin rpy="0 0 0" xyz="0 0 0"/>
+      <material name="blue" />
     </visual>
      <collision>
@@ -162,5 +168,5 @@
       <!-- <origin rpy="1.65 0 0" xyz="0.25 0.1 0.1"/> -->
       <origin rpy="1.6 0 0" xyz="0.05 0.1 -0.1"/>
-      <material name="blue" />
+      <material name="red"/>
     </visual>
     <collision>
@@ -259,5 +265,5 @@
         <clip>
           <near>0.02</near>
-          <far>8</far>
+          <far>80</far>
         </clip>
         <noise>
